Commit message: change link and joint naming conception

File: urdf/aleph2.urdf.xacro (robot description, xacro)
@@ -3,30 +3,73 @@
        name="aleph2">
   <xacro:include filename="$(find aleph2_description)/urdf/aleph2.gazebo" />
-  <material name="lazik">
-    <color rgba="0.3 0.3 0.3 1"/>
-  </material>
-  <material name="chromosom">
-    <color rgba="0 0 0.8 1"/>
-  </material>
-  <material name="kolo">
-    <texture filename="package://aleph_viz/textures/wheel.jpg" />
-  </material>
-  <material name="manip">
-    <color rgba="0.4 0.4 0.4 1"/>
-  </material>
-  <material name="maszt">
-    <color rgba="0.8 0.8 0.8 1" />
-  </material>
-  <xacro:macro name="chromosom" params="name">
-    <link name="chromosom_${name}">
+  <xacro:include filename="$(find aleph2_description)/urdf/materials.xacro" />
+  <link name="base_link">
+    <visual>
+      <geometry>
+        <mesh filename="package://aleph2_description/meshes/base.STL" />
+      </geometry>
+      <origin xyz="0 0 0" rpy="${pi/2} 0 ${pi/2}"/>
+      <material name="base" />
+    </visual>
+    <visual>
+      <geometry>
+        <cylinder radius="0.02" length="0.12" />
+      </geometry>
+      <origin xyz="0.06 0.125 0.063" />
+      <material name="motor">
+        <color rgba="0 0 0.5 1"/>
+      </material>
+    </visual>
+    <visual>
+      <geometry>
+        <cylinder radius="0.016" length="0.1" />
+      </geometry>
+      <origin xyz="0.151 0.175 0.053" />
+      <material name="encoder">
+        <color rgba="0 0.5 0 1"/>
+      </material>
+    </visual>
+    <collision>
+      <geometry>
+        <box size="0.72 0.5 0.1"/>
+      </geometry>
+      <origin xyz="-0.08 0 0"/>
+    </collision>
+    <collision>
+      <geometry>
+        <box size="0.16 0.5 0.1"/>
+      </geometry>
+      <origin xyz="-0.06 0 0.09"/>
+    </collision>
+    <collision>
+      <geometry>
+        <cylinder radius="0.02" length="0.12" />
+      </geometry>
+      <origin xyz="0.06 0.125 0.063" />
+    </collision>
+    <collision>
+      <geometry>
+        <cylinder radius="0.016" length="0.1" />
+      </geometry>
+      <origin xyz="0.151 0.175 0.053" />
+    </collision>
+    <inertial>
+      <origin xyz="-0.06700 0.00064 0.00551"/>
+      <mass value="9.0" />
+      <inertia ixx="0.23691" ixy="-0.00014" ixz="-0.00314"
+               iyy="0.23328" iyz="-0.00054" izz="0.40961" />
+    </inertial>
+  </link>
+  <xacro:macro name="rocker" params="name">
+    <link name="rocker_${name}_link">
       <visual>
         <geometry>
-          <mesh filename="package://aleph_viz/meshes/chromosom.STL"/>
+          <mesh filename="package://aleph2_description/meshes/rocker.STL"/>
         </geometry>
-        <material name="chromosom" />
+        <material name="rocker" />
       </visual>
       <collision>
         <geometry>
-          <mesh filename="package://aleph_viz/meshes/chromosom_collision.STL" />
+          <mesh filename="package://aleph2_description/meshes/rocker_collision.STL" />
         </geometry>
       </collision>
@@ -39,11 +82,11 @@
     </link>
   </xacro:macro>
-  <xacro:macro name="kolo" params="name">
-    <link name="kolo_${name}">
+  <xacro:macro name="wheel" params="name">
+    <link name="wheel_${name}_link">
       <visual>
         <geometry>
-          <mesh filename="package://aleph_viz/meshes/kolo.STL"/>
+          <mesh filename="package://aleph2_description/meshes/wheel.STL"/>
         </geometry>
-        <material name="kolo" />
+        <material name="wheel" />
       </visual>
       <visual>
@@ -85,77 +128,14 @@
     </link>
   </xacro:macro>
-  <link name="base_link">
-    <visual>
-      <geometry>
-        <mesh filename="package://aleph_viz/meshes/lazik.STL" />
-      </geometry>
-      <origin xyz="0 0 0" rpy="${pi/2} 0 ${pi/2}"/>
-      <material name="lazik" />
-    </visual>
-    <visual>
-      <geometry>
-        <cylinder radius="0.02" length="0.12" />
-      </geometry>
-      <origin xyz="0.06 0.125 0.063" />
-      <material name="silnik">
-        <color rgba="0 0 0.5 1"/>
-      </material>
-    </visual>
-    <visual>
-      <geometry>
-        <cylinder radius="0.016" length="0.1" />
-      </geometry>
-      <origin xyz="0.151 0.175 0.053" />
-      <material name="enkoder">
-        <color rgba="0 0.5 0 1"/>
-      </material>
-    </visual>
-    <collision>
-      <geometry>
-        <box size="0.72 0.5 0.1"/>
-      </geometry>
-      <origin xyz="-0.08 0 0"/>
-    </collision>
-    <collision>
-      <geometry>
-        <box size="0.16 0.5 0.1"/>
-      </geometry>
-      <origin xyz="-0.06 0 0.09"/>
-    </collision>
-    <collision>
-      <geometry>
-        <cylinder radius="0.02" length="0.12" />
-      </geometry>
-      <origin xyz="0.06 0.125 0.063" />
-    </collision>
-    <collision>
-      <geometry>
-        <cylinder radius="0.016" length="0.1" />
-      </geometry>
-      <origin xyz="0.151 0.175 0.053" />
-    </collision>
-    <inertial>
-      <origin xyz="-0.06700 0.00064 0.00551"/>
-      <mass value="9.0" />
-      <inertia ixx="0.23691" ixy="-0.00014" ixz="-0.00314"
-               iyy="0.23328" iyz="-0.00054" izz="0.40961" />
-    </inertial>
-  </link>
-  <xacro:chromosom name="R" />
-  <xacro:chromosom name="L" />
-  <xacro:kolo name="FR" />
-  <xacro:kolo name="RR" />
-  <xacro:kolo name="FL" />
-  <xacro:kolo name="RL" />
-  <!-- <link name="manip_support">
-    <inertial>
-      <mass value="0.0" />
-      <inertia ixx="1.0" ixy="0.0" ixz="0.0" iyy="1.0" iyz="0.0" izz="1.0" />
-    </inertial>
-  </link> -->
-  <link name="manip_base">
-    <visual>
-      <geometry>
-          <mesh filename="package://aleph_viz/meshes/A.STL"/>
+  <xacro:rocker name="R" />
+  <xacro:rocker name="L" />
+  <xacro:wheel name="FR" />
+  <xacro:wheel name="RR" />
+  <xacro:wheel name="FL" />
+  <xacro:wheel name="RL" />
+  <link name="manip_base_link">
+    <visual>
+      <geometry>
+          <mesh filename="package://aleph2_description/meshes/manip_base.STL"/>
       </geometry>
       <origin rpy="${pi/2} 0 ${-pi/2}"/>
@@ -193,8 +173,8 @@
     </inertial>
   </link>
-  <link name="manip_B">
-    <visual>
-      <geometry>
-          <mesh filename="package://aleph_viz/meshes/B.STL"/>
+  <link name="manip_shoulder_link">
+    <visual>
+      <geometry>
+          <mesh filename="package://aleph2_description/meshes/manip_shoulder.STL"/>
       </geometry>
       <origin rpy="${pi} 0 0"/>
@@ -206,5 +186,5 @@
       </geometry>
       <origin xyz="0.082 0 0.106" rpy="0 0 0" />
-      <material name="silnik">
+      <material name="motor">
         <color rgba="0 0 0.5 1"/>
       </material>
@@ -215,5 +195,5 @@
       </geometry>
       <origin xyz="0.2 0 0.106" rpy="0 0 0" />
-      <material name="silnik">
+      <material name="motor">
         <color rgba="0 0 0.5 1"/>
       </material>
@@ -259,5 +239,5 @@
       </geometry>
       <origin xyz="0.082 0 0.106" rpy="0 0 0" />
-      <material name="silnik">
+      <material name="motor">
         <color rgba="0 0 0.5 1"/>
       </material>
@@ -268,5 +248,5 @@
       </geometry>
       <origin xyz="0.2 0 0.106" rpy="0 0 0" />
-      <material name="silnik">
+      <material name="motor">
         <color rgba="0 0 0.5 1"/>
       </material>
@@ -297,8 +277,8 @@
     </inertial>
   </link>
-  <link name="manip_C">
-    <visual>
-      <geometry>
-          <mesh filename="package://aleph_viz/meshes/C.STL"/>
+  <link name="manip_elbow_link">
+    <visual>
+      <geometry>
+          <mesh filename="package://aleph2_description/meshes/manip_elbow.STL"/>
       </geometry>
       <origin rpy="0 ${pi/2} 0"/>
@@ -330,8 +310,8 @@
     </inertial>
   </link>
-  <link name="manip_D">
-    <visual>
-      <geometry>
-          <mesh filename="package://aleph_viz/meshes/D.STL"/>
+  <link name="manip_wrist_link">
+    <visual>
+      <geometry>
+          <mesh filename="package://aleph2_description/meshes/manip_wrist.STL"/>
       </geometry>
       <origin rpy="0 ${pi/2} 0"/>
@@ -343,5 +323,5 @@
       </geometry>
       <origin xyz="-0.03 0 0" rpy="0 ${pi/2} 0"/>
-      <material name="silnik">
+      <material name="motor">
         <color rgba="0 0 0.5 1"/>
       </material>
@@ -369,8 +349,8 @@
     </inertial>
   </link>
-  <link name="manip_efector">
-    <visual>
-      <geometry>
-          <mesh filename="package://aleph_viz/meshes/efector.STL"/>
+  <link name="manip_grasper_link">
+    <visual>
+      <geometry>
+          <mesh filename="package://aleph2_description/meshes/manip_grasper.STL"/>
       </geometry>
       <origin rpy="0 ${pi/2} 0"/>
@@ -402,8 +382,8 @@
     </inertial>
   </link>
-  <link name="manip_jaw_L">
-    <visual>
-      <geometry>
-        <mesh filename="package://aleph_viz/meshes/jaw.STL" />
+  <link name="manip_jaw_L_link">
+    <visual>
+      <geometry>
+        <mesh filename="package://aleph2_description/meshes/manip_jaw.STL" />
       </geometry>
       <origin rpy="${-pi/2} 0 ${pi/2}"/>
@@ -423,8 +403,8 @@
     </inertial>
   </link>
-  <link name="manip_jaw_R">
-    <visual>
-      <geometry>
-        <mesh filename="package://aleph_viz/meshes/jaw.STL" />
+  <link name="manip_jaw_R_link">
+    <visual>
+      <geometry>
+        <mesh filename="package://aleph2_description/meshes/manip_jaw.STL" />
       </geometry>
       <origin rpy="${-pi/2} ${pi} ${pi/2}"/>
@@ -444,6 +424,6 @@
     </inertial>
   </link>
-  <link name="efector_tip"/>
-  <link name="maszt">
+  <link name="manip_effector_tip_link"/>
+  <link name="mast_link">
     <visual>
       <geometry>
@@ -451,5 +431,5 @@
       </geometry>
       <origin xyz="0 0 0.65" rpi="0 0 0"/>
-      <material name="maszt" />
+      <material name="mast" />
     </visual>
     <collision>
@@ -474,5 +454,5 @@
       <origin xyz="0 0 0" rpy="0 0 0"/>
         <geometry>
-          <mesh filename="package://aleph_viz/meshes/ZED.stl" />
+          <mesh filename="package://aleph2_description/meshes/ZED.stl" />
         </geometry>
       <material name="light_grey">
@@ -485,127 +465,126 @@
       </geometry>
     </collision>
-    <inertial>
-      <mass value="1.0" />
-      <inertia ixx="1.0" ixy="0.0" ixz="0.0" iyy="1.0" iyz="0.0" izz="1.0" />
-    </inertial>
-  </link>
-  <!-- CHROMOSOMY -->
-  <joint name="chromosom_R_to_base" type="fixed">
+  </link>
+  <!-- ROCKERS -->
+  <joint name="rocker_R_joint" type="fixed">
     <parent link="base_link"/>
-    <child link="chromosom_R"/>
+    <child link="rocker_R_link"/>
       <origin xyz="0 -0.375 0" rpy="${pi/2} 0 ${pi}"/>
   </joint>
-  <joint name="chromosom_L_to_base" type="fixed">
+  <joint name="rocker_L_joint" type="fixed">
     <parent link="base_link"/>
-    <child link="chromosom_L"/>
+    <child link="rocker_L_link"/>
       <origin xyz="0 0.375 0" rpy="${pi/2} 0 0"/>
   </joint>
-  <!-- KOLA -->
-  <joint name="kolo_FR_to_chromosom_R" type="continuous">
-    <parent link="chromosom_R"/>
-    <child link="kolo_FR"/>
+  <!-- WHEELS -->
+  <joint name="wheel_FR_joint" type="continuous">
+    <parent link="rocker_R_link"/>
+    <child link="wheel_FR_link"/>
     <origin xyz="-0.418 -0.226 -0.07" rpy="${pi/2} 0 0" />
     <axis xyz="0 1 0"/>
-  </joint>
-  <joint name="kolo_RR_to_chromosom_R" type="continuous">
-    <parent link="chromosom_R"/>
-    <child link="kolo_RR"/>
+    <dynamics damping="0.0" friction="0.2"/>
+    <limit effort="1000" velocity="5.0"/>
+  </joint>
+  <joint name="wheel_RR_joint" type="continuous">
+    <parent link="rocker_R_link"/>
+    <child link="wheel_RR_link"/>
     <origin xyz="0.418 -0.226 -0.07" rpy="${-pi/2} 0 0" />
     <axis xyz="0 -1 0"/>
-  </joint>
-  <joint name="kolo_FL_to_chromosom_L" type="continuous">
-    <parent link="chromosom_L"/>
-    <child link="kolo_FL"/>
+    <dynamics damping="0.0" friction="0.2"/>
+    <limit effort="1000" velocity="5.0"/>
+  </joint>
+  <joint name="wheel_FL_joint" type="continuous">
+    <parent link="rocker_L_link"/>
+    <child link="wheel_FL_link"/>
     <origin xyz="0.418 -0.226 -0.07" rpy="${-pi/2} 0 0" />
     <axis xyz="0 1 0"/>
-  </joint>
-  <joint name="kolo_RL_to_chromosom_L" type="continuous">
-    <parent link="chromosom_L"/>
-    <child link="kolo_RL"/>
+    <dynamics damping="0.0" friction="0.2"/>
+    <limit effort="1000" velocity="5.0"/>
+  </joint>
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