Commit message: update gazebo references

File: urdf/aleph2.urdf.xacro (robot description, xacro)
@@ -586,140 +586,101 @@
     <origin xyz="0.265 -0.16 0.015"/>
   </joint>
-  <!-- <transmission name="kolo_FR_transmission">
-    <type>transmission_interface/SimpleTransmission</type>
-    <joint name="kolo_FR_to_chromosom_R">
-      <hardwareInterface>hardware_interface/VelocityJointInterface</hardwareInterface>
-    </joint>
-    <actuator name="kolo_FR_actuator">
-      <hardwareInterface>hardware_interface/VelocityJointInterface</hardwareInterface>
-      <mechanicalReduction>1</mechanicalReduction>
-    </actuator>
-  </transmission>
-  <transmission name="kolo_FL_transmission">
-    <type>transmission_interface/SimpleTransmission</type>
-    <joint name="kolo_FL_to_chromosom_L">
-      <hardwareInterface>hardware_interface/VelocityJointInterface</hardwareInterface>
-    </joint>
-    <actuator name="kolo_FL_actuator">
-      <hardwareInterface>hardware_interface/VelocityJointInterface</hardwareInterface>
-      <mechanicalReduction>1</mechanicalReduction>
-    </actuator>
-  </transmission>
-  <transmission name="kolo_RR_transmission">
-    <type>transmission_interface/SimpleTransmission</type>
-    <joint name="kolo_RR_to_chromosom_R">
-      <hardwareInterface>hardware_interface/VelocityJointInterface</hardwareInterface>
-    </joint>
-    <actuator name="kolo_RR_actuator">
-      <hardwareInterface>hardware_interface/VelocityJointInterface</hardwareInterface>
-      <mechanicalReduction>1</mechanicalReduction>
-    </actuator>
-  </transmission>
-  <transmission name="kolo_RL_transmission">
-    <type>transmission_interface/SimpleTransmission</type>
-    <joint name="kolo_RL_to_chromosom_L">
-      <hardwareInterface>hardware_interface/VelocityJointInterface</hardwareInterface>
-    </joint>
-    <actuator name="kolo_RL_actuator">
-      <hardwareInterface>hardware_interface/VelocityJointInterface</hardwareInterface>
-      <mechanicalReduction>1</mechanicalReduction>
-    </actuator>
-  </transmission> -->
-  <transmission name="kolo_FR_transmission">
-    <type>transmission_interface/SimpleTransmission</type>
-    <joint name="kolo_FR_to_chromosom_R">
-      <hardwareInterface>hardware_interface/EffortJointInterface</hardwareInterface>
-    </joint>
-    <actuator name="kolo_FR_actuator">
-      <hardwareInterface>hardware_interface/EffortJointInterface</hardwareInterface>
-      <mechanicalReduction>1</mechanicalReduction>
-    </actuator>
-  </transmission>
-  <transmission name="kolo_FL_transmission">
-    <type>transmission_interface/SimpleTransmission</type>
-    <joint name="kolo_FL_to_chromosom_L">
-      <hardwareInterface>hardware_interface/EffortJointInterface</hardwareInterface>
-    </joint>
-    <actuator name="kolo_FL_actuator">
-      <hardwareInterface>hardware_interface/EffortJointInterface</hardwareInterface>
-      <mechanicalReduction>1</mechanicalReduction>
-    </actuator>
-  </transmission>
-  <transmission name="kolo_RR_transmission">
-    <type>transmission_interface/SimpleTransmission</type>
-    <joint name="kolo_RR_to_chromosom_R">
-      <hardwareInterface>hardware_interface/EffortJointInterface</hardwareInterface>
-    </joint>
-    <actuator name="kolo_RR_actuator">
-      <hardwareInterface>hardware_interface/EffortJointInterface</hardwareInterface>
-      <mechanicalReduction>1</mechanicalReduction>
-    </actuator>
-  </transmission>
-  <transmission name="kolo_RL_transmission">
-    <type>transmission_interface/SimpleTransmission</type>
-    <joint name="kolo_RL_to_chromosom_L">
-      <hardwareInterface>hardware_interface/EffortJointInterface</hardwareInterface>
-    </joint>
-    <actuator name="kolo_RL_actuator">
-      <hardwareInterface>hardware_interface/EffortJointInterface</hardwareInterface>
-      <mechanicalReduction>1</mechanicalReduction>
-    </actuator>
-  </transmission>
-  <transmission name="base_to_frame_transmission">
-    <type>transmission_interface/SimpleTransmission</type>
-    <joint name="base_to_frame">
-      <hardwareInterface>hardware_interface/EffortJointInterface</hardwareInterface>
-    </joint>
-    <actuator name="base_to_frame_actuator">
-      <hardwareInterface>hardware_interface/EffortJointInterface</hardwareInterface>
-      <mechanicalReduction>1</mechanicalReduction>
-    </actuator>
-  </transmission>
-  <transmission name="B_to_base_transmission">
-    <type>transmission_interface/SimpleTransmission</type>
-    <joint name="B_to_base">
-      <hardwareInterface>hardware_interface/EffortJointInterface</hardwareInterface>
-    </joint>
-    <actuator name="B_to_base_actuator">
-      <hardwareInterface>hardware_interface/EffortJointInterface</hardwareInterface>
-      <mechanicalReduction>1</mechanicalReduction>
-    </actuator>
-  </transmission>
-  <transmission name="C_to_B_transmission">
-    <type>transmission_interface/SimpleTransmission</type>
-    <joint name="C_to_B">
-      <hardwareInterface>hardware_interface/EffortJointInterface</hardwareInterface>
-    </joint>
-    <actuator name="C_to_B_actuator">
-      <hardwareInterface>hardware_interface/EffortJointInterface</hardwareInterface>
-      <mechanicalReduction>1</mechanicalReduction>
-    </actuator>
-  </transmission>
-  <transmission name="efector_to_C_transmission">
-    <type>transmission_interface/SimpleTransmission</type>
-    <joint name="efector_to_C">
-      <hardwareInterface>hardware_interface/EffortJointInterface</hardwareInterface>
-    </joint>
-    <actuator name="efector_to_C_actuator">
-      <hardwareInterface>hardware_interface/EffortJointInterface</hardwareInterface>
-      <mechanicalReduction>1</mechanicalReduction>
-    </actuator>
-  </transmission>
-  <transmission name="efector_roll_transmission">
-    <type>transmission_interface/SimpleTransmission</type>
-    <joint name="efector_roll">
-      <hardwareInterface>hardware_interface/EffortJointInterface</hardwareInterface>
-    </joint>
-    <actuator name="efector_roll_actuator">
-      <hardwareInterface>hardware_interface/EffortJointInterface</hardwareInterface>
-      <mechanicalReduction>1</mechanicalReduction>
-    </actuator>
-  </transmission>
-  <transmission name="efector_grip_transmission">
-    <type>transmission_interface/SimpleTransmission</type>
-    <joint name="efector_grip">
-      <hardwareInterface>hardware_interface/EffortJointInterface</hardwareInterface>
-    </joint>
-    <actuator name="efector_grip_actuator">
+  <!-- TRASNMISSIONS -->
+  <transmission name="wheel_FR_transmission">
+    <type>transmission_interface/SimpleTransmission</type>
+    <joint name="wheel_FR_joint">
+      <hardwareInterface>hardware_interface/EffortJointInterface</hardwareInterface>
+    </joint>
+    <actuator name="wheel_FR_actuator">
+      <hardwareInterface>hardware_interface/EffortJointInterface</hardwareInterface>
+      <mechanicalReduction>1</mechanicalReduction>
+    </actuator>
+  </transmission>
+  <transmission name="wheel_FL_transmission">
+    <type>transmission_interface/SimpleTransmission</type>
+    <joint name="wheel_FL_joint">
+      <hardwareInterface>hardware_interface/EffortJointInterface</hardwareInterface>
+    </joint>
+    <actuator name="wheel_FL_actuator">
+      <hardwareInterface>hardware_interface/EffortJointInterface</hardwareInterface>
+      <mechanicalReduction>1</mechanicalReduction>
+    </actuator>
+  </transmission>
+  <transmission name="wheel_RR_transmission">
+    <type>transmission_interface/SimpleTransmission</type>
+    <joint name="wheel_RR_joint">
+      <hardwareInterface>hardware_interface/EffortJointInterface</hardwareInterface>
+    </joint>
+    <actuator name="wheel_RR_actuator">
+      <hardwareInterface>hardware_interface/EffortJointInterface</hardwareInterface>
+      <mechanicalReduction>1</mechanicalReduction>
+    </actuator>
+  </transmission>
+  <transmission name="wheel_RL_transmission">
+    <type>transmission_interface/SimpleTransmission</type>
+    <joint name="wheel_RL_joint">
+      <hardwareInterface>hardware_interface/EffortJointInterface</hardwareInterface>
+    </joint>
+    <actuator name="wheel_RL_actuator">
+      <hardwareInterface>hardware_interface/EffortJointInterface</hardwareInterface>
+      <mechanicalReduction>1</mechanicalReduction>
+    </actuator>
+  </transmission>
+  <transmission name="manip_base_transmission">
+    <type>transmission_interface/SimpleTransmission</type>
+    <joint name="manip_base_joint">
+      <hardwareInterface>hardware_interface/EffortJointInterface</hardwareInterface>
+    </joint>
+    <actuator name="manip_base_actuator">
+      <hardwareInterface>hardware_interface/EffortJointInterface</hardwareInterface>
+      <mechanicalReduction>1</mechanicalReduction>
+    </actuator>
+  </transmission>
+  <transmission name="manip_shoulder_transmission">
+    <type>transmission_interface/SimpleTransmission</type>
+    <joint name="manip_shoulder_joint">
+      <hardwareInterface>hardware_interface/EffortJointInterface</hardwareInterface>
+    </joint>
+    <actuator name="manip_shoulder_actuator">
+      <hardwareInterface>hardware_interface/EffortJointInterface</hardwareInterface>
+      <mechanicalReduction>1</mechanicalReduction>
+    </actuator>
+  </transmission>
+  <transmission name="manip_elbow_transmission">
+    <type>transmission_interface/SimpleTransmission</type>
+    <joint name="manip_elbow_joint">
+      <hardwareInterface>hardware_interface/EffortJointInterface</hardwareInterface>
+    </joint>
+    <actuator name="manip_elbow_actuator">
+      <hardwareInterface>hardware_interface/EffortJointInterface</hardwareInterface>
+      <mechanicalReduction>1</mechanicalReduction>
+    </actuator>
+  </transmission>
+  <transmission name="manip_wrist_transmission">
+    <type>transmission_interface/SimpleTransmission</type>
+    <joint name="manip_wrist_joint">
+      <hardwareInterface>hardware_interface/EffortJointInterface</hardwareInterface>
+    </joint>
+    <actuator name="manip_wrist_actuator">
+      <hardwareInterface>hardware_interface/EffortJointInterface</hardwareInterface>
+      <mechanicalReduction>1</mechanicalReduction>
+    </actuator>
+  </transmission>
+  <transmission name="manip_grasper_transmission">
+    <type>transmission_interface/SimpleTransmission</type>
+    <joint name="manip_grasper_joint">
+      <hardwareInterface>hardware_interface/EffortJointInterface</hardwareInterface>
+    </joint>
+    <actuator name="manip_grasper_actuator">
+      <hardwareInterface>hardware_interface/EffortJointInterface</hardwareInterface>
+      <mechanicalReduction>1</mechanicalReduction>
+    </actuator>
+  </transmission>
+  <transmission name="manip_grip_transmission">
+    <type>transmission_interface/SimpleTransmission</type>
+    <joint name="manip_grip_joint">
+      <hardwareInterface>hardware_interface/EffortJointInterface</hardwareInterface>
+    </joint>
+    <actuator name="manip_grip_actuator">
       <hardwareInterface>hardware_interface/EffortJointInterface</hardwareInterface>
       <mechanicalReduction>1</mechanicalReduction>

Commit message: rename grasper to gripper

File: urdf/aleph2.urdf.xacro (robot description, xacro)
@@ -349,8 +349,8 @@
     </inertial>
   </link>
-  <link name="manip_grasper_link">
-    <visual>
-      <geometry>
-          <mesh filename="package://aleph2_description/meshes/manip_grasper.STL"/>
+  <link name="manip_gripper_link">
+    <visual>
+      <geometry>
+          <mesh filename="package://aleph2_description/meshes/manip_gripper.STL"/>
       </geometry>
       <origin rpy="0 ${pi/2} 0"/>
@@ -535,5 +535,5 @@
     <dynamics damping="0.0" friction="0.1"/>
   </joint>
-  <joint name="manip_wrist_joint" type="revolute">
+  <joint name="manip_wrist_tilt_joint" type="revolute">
     <parent link="manip_elbow_link"/>
     <child link="manip_wrist_link"/>
@@ -543,7 +543,7 @@
     <dynamics damping="0.0" friction="0.1"/>
   </joint>
-  <joint name="manip_grasper_joint" type="revolute">
+  <joint name="manip_wrist_roll_joint" type="revolute">
     <parent link="manip_wrist_link"/>
-    <child link="manip_grasper_link"/>
+    <child link="manip_gripper_link"/>
     <origin xyz="0.06 0 0" rpy="${-pi/2} 0 0"/>
     <axis xyz="-1 0 0" />
@@ -551,6 +551,6 @@
     <dynamics damping="0.0" friction="0.1"/>
   </joint>
-  <joint name="manip_grip_joint" type="prismatic">
-    <parent link="manip_grasper_link"/>
+  <joint name="manip_gripper_joint" type="prismatic">
+    <parent link="manip_gripper_link"/>
     <child link="manip_jaw_L_link"/>
     <origin xyz="0.025 -0.03 0"/>
@@ -559,15 +559,15 @@
     <dynamics damping="0.0" friction="0.1"/>
   </joint>
-  <joint name="manip_grip_joint_mimic" type="prismatic">
-    <parent link="manip_grasper_link"/>
+  <joint name="manip_gripper_joint_mimic" type="prismatic">
+    <parent link="manip_gripper_link"/>
     <child link="manip_jaw_R_link"/>
     <origin xyz="0.025 0.03 0"/>
     <axis xyz="0 -1 0" />
-    <mimic joint="manip_grip_joint" />
+    <mimic joint="manip_gripper_joint" />
     <limit effort="150" lower="-0.033" upper="0" velocity="0.05"/>
     <dynamics damping="0.0" friction="0.1"/>
   </joint>
   <joint name="manip_effector_tip_joint" type="fixed">
-    <parent link="manip_grasper_link"/>
+    <parent link="manip_gripper_link"/>
     <child link="manip_effector_tip_link"/>
     <origin xyz="0.20 0 0"/>
@@ -657,30 +657,30 @@
     </actuator>
   </transmission>
-  <transmission name="manip_wrist_transmission">
-    <type>transmission_interface/SimpleTransmission</type>
-    <joint name="manip_wrist_joint">
-      <hardwareInterface>hardware_interface/EffortJointInterface</hardwareInterface>
-    </joint>
-    <actuator name="manip_wrist_actuator">
-      <hardwareInterface>hardware_interface/EffortJointInterface</hardwareInterface>
-      <mechanicalReduction>1</mechanicalReduction>
-    </actuator>
-  </transmission>
-  <transmission name="manip_grasper_transmission">
-    <type>transmission_interface/SimpleTransmission</type>
-    <joint name="manip_grasper_joint">
-      <hardwareInterface>hardware_interface/EffortJointInterface</hardwareInterface>
-    </joint>
-    <actuator name="manip_grasper_actuator">
-      <hardwareInterface>hardware_interface/EffortJointInterface</hardwareInterface>
-      <mechanicalReduction>1</mechanicalReduction>
-    </actuator>
-  </transmission>
-  <transmission name="manip_grip_transmission">
-    <type>transmission_interface/SimpleTransmission</type>
-    <joint name="manip_grip_joint">
-      <hardwareInterface>hardware_interface/EffortJointInterface</hardwareInterface>
-    </joint>
-    <actuator name="manip_grip_actuator">
+  <transmission name="manip_wrist_tilt_transmission">
+    <type>transmission_interface/SimpleTransmission</type>
+    <joint name="manip_wrist_tilt_joint">
+      <hardwareInterface>hardware_interface/EffortJointInterface</hardwareInterface>
+    </joint>
+    <actuator name="manip_wrist_tilt_actuator">
+      <hardwareInterface>hardware_interface/EffortJointInterface</hardwareInterface>
+      <mechanicalReduction>1</mechanicalReduction>
+    </actuator>
+  </transmission>
+  <transmission name="manip_wrist_roll_transmission">
+    <type>transmission_interface/SimpleTransmission</type>
+    <joint name="manip_wrist_roll_joint">
+      <hardwareInterface>hardware_interface/EffortJointInterface</hardwareInterface>
+    </joint>
+    <actuator name="manip_wrist_roll_actuator">
+      <hardwareInterface>hardware_interface/EffortJointInterface</hardwareInterface>
+      <mechanicalReduction>1</mechanicalReduction>
+    </actuator>
+  </transmission>
+  <transmission name="manip_gripper_transmission">
+    <type>transmission_interface/SimpleTransmission</type>
+    <joint name="manip_gripper_joint">
+      <hardwareInterface>hardware_interface/EffortJointInterface</hardwareInterface>
+    </joint>
+    <actuator name="manip_gripper_actuator">
       <hardwareInterface>hardware_interface/EffortJointInterface</hardwareInterface>
       <mechanicalReduction>1</mechanicalReduction>

Commit message: modify wheel parameters

File: urdf/aleph2.urdf.xacro (robot description, xacro)
@@ -483,6 +483,6 @@
     <origin xyz="-0.418 -0.226 -0.07" rpy="${pi/2} 0 0" />
     <axis xyz="0 1 0"/>
-    <dynamics damping="0.0" friction="0.2"/>
-    <limit effort="1000" velocity="5.0"/>
+    <dynamics damping="0.5" friction="0.2"/>
+    <limit effort="20" velocity="25.0"/>
   </joint>
   <joint name="wheel_RR_joint" type="continuous">
@@ -491,6 +491,6 @@
     <origin xyz="0.418 -0.226 -0.07" rpy="${-pi/2} 0 0" />
     <axis xyz="0 -1 0"/>
-    <dynamics damping="0.0" friction="0.2"/>
-    <limit effort="1000" velocity="5.0"/>
+    <dynamics damping="0.5" friction="0.2"/>
+    <limit effort="20" velocity="25.0"/>
   </joint>
   <joint name="wheel_FL_joint" type="continuous">
@@ -499,6 +499,6 @@
     <origin xyz="0.418 -0.226 -0.07" rpy="${-pi/2} 0 0" />
     <axis xyz="0 1 0"/>
-    <dynamics damping="0.0" friction="0.2"/>
-    <limit effort="1000" velocity="5.0"/>
+    <dynamics damping="0.5" friction="0.2"/>
+    <limit effort="20" velocity="25.0"/>
   </joint>
   <joint name="wheel_RL_joint" type="continuous">
@@ -507,6 +507,6 @@
     <origin xyz="-0.418 -0.226 -0.07" rpy="${pi/2} 0 0" />
     <axis xyz="0 -1 0"/>
-    <dynamics damping="0.0" friction="0.2"/>
-    <limit effort="1000" velocity="5.0"/>
+    <dynamics damping="0.5" friction="0.2"/>
+    <limit effort="20" velocity="25.0"/>
   </joint>
   <!-- MANIP -->
@@ -590,8 +590,8 @@
     <type>transmission_interface/SimpleTransmission</type>
     <joint name="wheel_FR_joint">
-      <hardwareInterface>hardware_interface/EffortJointInterface</hardwareInterface>
+      <hardwareInterface>hardware_interface/VelocityJointInterface</hardwareInterface>
     </joint>
     <actuator name="wheel_FR_actuator">
-      <hardwareInterface>hardware_interface/EffortJointInterface</hardwareInterface>
+      <hardwareInterface>hardware_interface/VelocityJointInterface</hardwareInterface>
       <mechanicalReduction>1</mechanicalReduction>
     </actuator>
@@ -600,8 +600,8 @@
     <type>transmission_interface/SimpleTransmission</type>
     <joint name="wheel_FL_joint">
-      <hardwareInterface>hardware_interface/EffortJointInterface</hardwareInterface>
+      <hardwareInterface>hardware_interface/VelocityJointInterface</hardwareInterface>
     </joint>
     <actuator name="wheel_FL_actuator">
-      <hardwareInterface>hardware_interface/EffortJointInterface</hardwareInterface>
+      <hardwareInterface>hardware_interface/VelocityJointInterface</hardwareInterface>
       <mechanicalReduction>1</mechanicalReduction>
     </actuator>
@@ -610,8 +610,8 @@
     <type>transmission_interface/SimpleTransmission</type>
     <joint name="wheel_RR_joint">
-      <hardwareInterface>hardware_interface/EffortJointInterface</hardwareInterface>
+      <hardwareInterface>hardware_interface/VelocityJointInterface</hardwareInterface>
     </joint>
     <actuator name="wheel_RR_actuator">
-      <hardwareInterface>hardware_interface/EffortJointInterface</hardwareInterface>
+      <hardwareInterface>hardware_interface/VelocityJointInterface</hardwareInterface>
       <mechanicalReduction>1</mechanicalReduction>
     </actuator>
@@ -620,8 +620,8 @@
     <type>transmission_interface/SimpleTransmission</type>
     <joint name="wheel_RL_joint">
-      <hardwareInterface>hardware_interface/EffortJointInterface</hardwareInterface>
+      <hardwareInterface>hardware_interface/VelocityJointInterface</hardwareInterface>
     </joint>
     <actuator name="wheel_RL_actuator">
-      <hardwareInterface>hardware_interface/EffortJointInterface</hardwareInterface>
+      <hardwareInterface>hardware_interface/VelocityJointInterface</hardwareInterface>
       <mechanicalReduction>1</mechanicalReduction>
     </actuator>

Commit message: update wheel radius, change shoulder origin

File: urdf/aleph2.urdf.xacro (robot description, xacro)
@@ -110,5 +110,5 @@
       <collision>
         <geometry>
-          <cylinder radius="0.18" length="0.1" />
+          <cylinder radius="0.16" length="0.1" />
         </geometry>
         <origin xyz="0 0 0" rpy="${pi/2} 0 0"/>
@@ -522,8 +522,8 @@
     <parent link="manip_base_link"/>
     <child link="manip_shoulder_link"/>
-    <origin xyz="0 0 0.09" rpy="${pi/2} 0 0"/>
+    <origin xyz="0 0 0.09" rpy="${pi/2} ${-pi/2} 0"/>
     <axis xyz="0 0 1" />
-    <limit effort="32000" lower="0.0" upper="${pi}" velocity="0.3"/>
-    <dynamics damping="0.0" friction="0.1"/>
+    <limit effort="32000" lower="${-pi/2}" upper="${pi/2}" velocity="0.3"/>
+    <dynamics damping="0.0" friction="50.0"/>
   </joint>
   <joint name="manip_elbow_joint" type="revolute">
