Commit message: Poprawki tarć w gazebo

File: urdf/aleph2.urdf.xacro (robot description, xacro)
@@ -517,5 +517,5 @@
     <axis xyz="0 0 1"/>
     <limit effort="32000" velocity="0.15"/>
-    <dynamics damping="0.0" friction="0.1"/>
+    <dynamics damping="100.0" friction="60.0"/>
   </joint>
   <joint name="manip_shoulder_joint" type="revolute">
@@ -524,6 +524,6 @@
     <origin xyz="0 0 0.09" rpy="${pi/2} ${-pi/2} 0"/>
     <axis xyz="0 0 1" />
-    <limit effort="32000" lower="${-pi/2}" upper="${pi/2}" velocity="0.3"/>
-    <dynamics damping="0.0" friction="50.0"/>
+    <limit effort="320" lower="${-pi/2}" upper="${pi/2}" velocity="0.3"/>
+    <dynamics damping="100.0" friction="60.0"/>
   </joint>
   <joint name="manip_elbow_joint" type="revolute">
@@ -532,6 +532,6 @@
     <origin xyz="0.4 0 0" rpy="${pi} 0 0" />
     <axis xyz="0 0 -1" />
-    <limit effort="32000" lower="-2.28" upper="2.43" velocity="0.5"/>
-    <dynamics damping="0.0" friction="0.1"/>
+    <limit effort="320" lower="-2.28" upper="2.43" velocity="0.5"/>
+    <dynamics damping="100.0" friction="50.0"/>
   </joint>
   <joint name="manip_wrist_tilt_joint" type="revolute">
@@ -540,6 +540,6 @@
     <origin xyz="0.4 0 0" />
     <axis xyz="0 0 -1" />
-    <limit effort="32000" lower="-2.2" upper="2.2" velocity="0.5"/>
-    <dynamics damping="0.0" friction="0.1"/>
+    <limit effort="320" lower="-2.2" upper="2.2" velocity="0.5"/>
+    <dynamics damping="90.0" friction="40.0"/>
   </joint>
   <joint name="manip_wrist_roll_joint" type="revolute">
@@ -548,6 +548,6 @@
     <origin xyz="0.06 0 0" rpy="${-pi/2} 0 0"/>
     <axis xyz="-1 0 0" />
-    <limit effort="32000" lower="${-pi}" upper="${pi}" velocity="0.5"/>
-    <dynamics damping="0.0" friction="0.1"/>
+    <limit effort="320" lower="${-pi}" upper="${pi}" velocity="0.5"/>
+    <dynamics damping="3.0" friction="10.0"/>
   </joint>
   <joint name="manip_gripper_joint" type="prismatic">
@@ -557,5 +557,5 @@
     <axis xyz="0 1 0" />
     <limit effort="150" lower="-0.033" upper="0" velocity="0.05"/>
-    <dynamics damping="0.0" friction="0.1"/>
+    <dynamics damping="5.0" friction="0.1"/>
   </joint>
   <joint name="manip_gripper_joint_mimic" type="prismatic">
@@ -566,5 +566,5 @@
     <mimic joint="manip_gripper_joint" />
     <limit effort="150" lower="-0.033" upper="0" velocity="0.05"/>
-    <dynamics damping="0.0" friction="0.1"/>
+    <dynamics damping="5.0" friction="0.1"/>
   </joint>
   <joint name="manip_effector_tip_joint" type="fixed">

Commit message: add names to visual tags in wheel links

File: urdf/aleph2.urdf.xacro (robot description, xacro)
@@ -90,5 +90,5 @@
         <material name="wheel" />
       </visual>
-      <visual>
+      <visual name="piasta">
         <geometry>
           <cylinder radius="0.05" length="0.12"/>
@@ -99,5 +99,5 @@
         </material>
       </visual>
-      <visual>
+      <visual name="walek">
         <geometry>
           <cylinder radius="0.0055" length="0.15"/>

Commit message: update some physical properties, robot NO LONGER EXPLODES in Gazebo

File: urdf/aleph2.urdf.xacro (robot description, xacro)
@@ -516,5 +516,5 @@
     <origin xyz="0.151 0.0035 0.032"/>
     <axis xyz="0 0 1"/>
-    <limit effort="32000" velocity="0.15"/>
+    <limit effort="100" velocity="0.15"/>
     <dynamics damping="100.0" friction="60.0"/>
   </joint>
@@ -524,5 +524,5 @@
     <origin xyz="0 0 0.09" rpy="${pi/2} ${-pi/2} 0"/>
     <axis xyz="0 0 1" />
-    <limit effort="320" lower="${-pi/2}" upper="${pi/2}" velocity="0.3"/>
+    <limit effort="100" lower="${-pi/2}" upper="${pi/2}" velocity="0.3"/>
     <dynamics damping="100.0" friction="60.0"/>
   </joint>
@@ -532,5 +532,5 @@
     <origin xyz="0.4 0 0" rpy="${pi} 0 0" />
     <axis xyz="0 0 -1" />
-    <limit effort="320" lower="-2.28" upper="2.43" velocity="0.5"/>
+    <limit effort="100" lower="-2.28" upper="2.43" velocity="0.5"/>
     <dynamics damping="100.0" friction="50.0"/>
   </joint>
@@ -540,6 +540,6 @@
     <origin xyz="0.4 0 0" />
     <axis xyz="0 0 -1" />
-    <limit effort="320" lower="-2.2" upper="2.2" velocity="0.5"/>
-    <dynamics damping="90.0" friction="40.0"/>
+    <limit effort="100" lower="-2.2" upper="2.2" velocity="0.5"/>
+    <dynamics damping="20.0" friction="40.0"/>
   </joint>
   <joint name="manip_wrist_roll_joint" type="revolute">
@@ -548,5 +548,5 @@
     <origin xyz="0.06 0 0" rpy="${-pi/2} 0 0"/>
     <axis xyz="-1 0 0" />
-    <limit effort="320" lower="${-pi}" upper="${pi}" velocity="0.5"/>
+    <limit effort="50" lower="${-pi}" upper="${pi}" velocity="0.5"/>
     <dynamics damping="3.0" friction="10.0"/>
   </joint>
@@ -556,6 +556,6 @@
     <origin xyz="0.025 -0.03 0"/>
     <axis xyz="0 1 0" />
-    <limit effort="150" lower="-0.033" upper="0" velocity="0.05"/>
-    <dynamics damping="5.0" friction="0.1"/>
+    <limit effort="60" lower="-0.033" upper="0" velocity="0.05"/>
+    <dynamics damping="5.0" friction="30.0"/>
   </joint>
   <joint name="manip_gripper_joint_mimic" type="prismatic">
@@ -565,6 +565,6 @@
     <axis xyz="0 -1 0" />
     <mimic joint="manip_gripper_joint" />
-    <limit effort="150" lower="-0.033" upper="0" velocity="0.05"/>
-    <dynamics damping="5.0" friction="0.1"/>
+    <limit effort="60" lower="-0.033" upper="0" velocity="0.05"/>
+    <dynamics damping="5.0" friction="30.0"/>
   </joint>
   <joint name="manip_effector_tip_joint" type="fixed">
@@ -572,5 +572,4 @@
     <child link="manip_effector_tip_link"/>
     <origin xyz="0.20 0 0"/>
-    <dynamics damping="0.0" friction="0.1"/>
   </joint>
   <!-- MASZT -->
