Commit message: aleph2_description: Move drivetrain to separate URDF file, add rockers_fixed argument

File: aleph2_description/urdf/aleph2.urdf.xacro (robot description, xacro)
@@ -3,8 +3,10 @@
        name="aleph2">
   <xacro:arg name="fixed" default="false"/>
-  <xacro:include filename="$(find aleph2_description)/urdf/aleph2.gazebo.xacro" />
-  <xacro:include filename="$(find aleph2_description)/urdf/materials.urdf.xacro" />
-  <xacro:include filename="$(find aleph2_description)/urdf/manip.urdf.xacro" />
-  <xacro:include filename="$(find aleph2_description)/urdf/zed.urdf.xacro" />
+  <xacro:arg name="rockers_fixed" default="true"/>
+  <xacro:include filename="$(find aleph2_description)/urdf/include/materials.urdf.xacro" />
+  <xacro:include filename="$(find aleph2_description)/urdf/include/aleph2.gazebo.xacro" />
+  <xacro:include filename="$(find aleph2_description)/urdf/include/drivetrain.urdf.xacro" />
+  <xacro:include filename="$(find aleph2_description)/urdf/include/manip.urdf.xacro" />
+  <xacro:include filename="$(find aleph2_description)/urdf/include/zed.urdf.xacro" />
   <xacro:if value="$(arg fixed)">
     <link name="world"/>
@@ -94,56 +96,6 @@
     </link>
   </xacro:macro>
-  <xacro:macro name="wheel" params="name">
-    <link name="wheel_${name}_link">
-      <visual>
-        <geometry>
-          <mesh filename="package://aleph2_description/meshes/wheel.STL"/>
-        </geometry>
-        <material name="wheel" />
-      </visual>
-      <visual name="piasta">
-        <geometry>
-          <cylinder radius="0.05" length="0.12"/>
-        </geometry>
-        <origin xyz="0 0 0" rpy="${pi/2} 0 0"/>
-        <material name="piasta">
-          <color rgba="0.5 0.5 0.5 1" />
-        </material>
-      </visual>
-      <visual name="walek">
-        <geometry>
-          <cylinder radius="0.0055" length="0.15"/>
-        </geometry>
-        <origin xyz="0 0 0" rpy="${pi/2} 0 0"/>
-        <material name="walek">
-          <color rgba="0.7 0.7 0.7 1" />
-        </material>
-      </visual>
-      <collision>
-        <geometry>
-          <cylinder radius="0.16" length="0.1" />
-        </geometry>
-        <origin xyz="0 0 0" rpy="${pi/2} 0 0"/>
-      </collision>
-      <collision>
-        <geometry>
-          <cylinder radius="0.007" length="0.15"/>
-        </geometry>
-        <origin xyz="0 0 0" rpy="${pi/2} 0 0"/>
-      </collision>
-      <inertial>
-        <origin xyz="0.00000 0.00000 0.00000"/>
-        <mass value="6.0" />
-        <inertia ixx="0.03845" ixy="0.00000" ixz="0.00000"
-                 iyy="0.06495" iyz="0.00000" izz="0.03845" />
-      </inertial>
-    </link>
-  </xacro:macro>
   <xacro:rocker name="R" />
   <xacro:rocker name="L" />
-  <xacro:wheel name="FR" />
-  <xacro:wheel name="RR" />
-  <xacro:wheel name="FL" />
-  <xacro:wheel name="RL" />
   <link name="mast_link">
     <visual>
@@ -172,13 +124,25 @@
   </link>
   <!-- JOINTS -->
-  <joint name="rocker_R_joint" type="fixed">
+  <xacro:if value="$(arg rockers_fixed)">
+    <xacro:property name="rockers_joint_type" value="fixed"/>
+  </xacro:if>
+  <xacro:unless value="$(arg rockers_fixed)">
+    <xacro:property name="rockers_joint_type" value="revolute"/>
+  </xacro:unless>
+  <joint name="rocker_R_joint" type="${rockers_joint_type}">
     <parent link="base_link"/>
     <child link="rocker_R_link"/>
-      <origin xyz="0 -0.375 0" rpy="${pi/2} 0 ${pi}"/>
+    <origin xyz="0 -0.375 0" rpy="${pi/2} 0 ${pi}"/>
+    <axis xyz="0 0 1"/>
+    <limit effort="100.0" lower="-0.3" upper="0.3" velocity="100.0"/>
+    <dynamics friction="1.0" damping="0.1"/>
   </joint>
-  <joint name="rocker_L_joint" type="fixed">
+  <joint name="rocker_L_joint" type="${rockers_joint_type}">
     <parent link="base_link"/>
     <child link="rocker_L_link"/>
-      <origin xyz="0 0.375 0" rpy="${pi/2} 0 0"/>
+    <origin xyz="0 0.375 0" rpy="${pi/2} 0 0"/>
+    <axis xyz="0 0 1"/>
+    <limit effort="100.0" lower="-0.3" upper="0.3" velocity="100.0"/>
+    <dynamics friction="1.0" damping="0.1"/>
   </joint>
   <joint name="mast_joint" type="fixed">
@@ -187,76 +151,3 @@
     <origin xyz="-0.22 0.25 -0.15"/>
   </joint>
-  <joint name="wheel_FR_joint" type="continuous">
-    <parent link="rocker_R_link"/>
-    <child link="wheel_FR_link"/>
-    <origin xyz="-0.418 -0.226 -0.07" rpy="${pi/2} 0 0" />
-    <axis xyz="0 1 0"/>
-    <dynamics damping="0.5" friction="0.2"/>
-    <limit effort="20" velocity="25.0"/>
-  </joint>
-  <joint name="wheel_RR_joint" type="continuous">
-    <parent link="rocker_R_link"/>
-    <child link="wheel_RR_link"/>
-    <origin xyz="0.418 -0.226 -0.07" rpy="${-pi/2} 0 0" />
-    <axis xyz="0 -1 0"/>
-    <dynamics damping="0.5" friction="0.2"/>
-    <limit effort="20" velocity="25.0"/>
-  </joint>
-  <joint name="wheel_FL_joint" type="continuous">
-    <parent link="rocker_L_link"/>
-    <child link="wheel_FL_link"/>
-    <origin xyz="0.418 -0.226 -0.07" rpy="${-pi/2} 0 0" />
-    <axis xyz="0 1 0"/>
-    <dynamics damping="0.5" friction="0.2"/>
-    <limit effort="20" velocity="25.0"/>
-  </joint>
-  <joint name="wheel_RL_joint" type="continuous">
-    <parent link="rocker_L_link"/>
-    <child link="wheel_RL_link"/>
-    <origin xyz="-0.418 -0.226 -0.07" rpy="${pi/2} 0 0" />
-    <axis xyz="0 -1 0"/>
-    <dynamics damping="0.5" friction="0.2"/>
-    <limit effort="20" velocity="25.0"/>
-  </joint>
-  <!-- TRASNMISSIONS -->
-  <transmission name="wheel_FR_transmission">
-    <type>transmission_interface/SimpleTransmission</type>
-    <joint name="wheel_FR_joint">
-      <hardwareInterface>hardware_interface/VelocityJointInterface</hardwareInterface>
-    </joint>
-    <actuator name="wheel_FR_actuator">
-      <hardwareInterface>hardware_interface/VelocityJointInterface</hardwareInterface>
-      <mechanicalReduction>1</mechanicalReduction>
-    </actuator>
-  </transmission>
-  <transmission name="wheel_FL_transmission">
-    <type>transmission_interface/SimpleTransmission</type>
-    <joint name="wheel_FL_joint">
-      <hardwareInterface>hardware_interface/VelocityJointInterface</hardwareInterface>
-    </joint>
-    <actuator name="wheel_FL_actuator">
-      <hardwareInterface>hardware_interface/VelocityJointInterface</hardwareInterface>
-      <mechanicalReduction>1</mechanicalReduction>
-    </actuator>
-  </transmission>
-  <transmission name="wheel_RR_transmission">
-    <type>transmission_interface/SimpleTransmission</type>
-    <joint name="wheel_RR_joint">
-      <hardwareInterface>hardware_interface/VelocityJointInterface</hardwareInterface>
-    </joint>
-    <actuator name="wheel_RR_actuator">
-      <hardwareInterface>hardware_interface/VelocityJointInterface</hardwareInterface>
-      <mechanicalReduction>1</mechanicalReduction>
-    </actuator>
-  </transmission>
-  <transmission name="wheel_RL_transmission">
-    <type>transmission_interface/SimpleTransmission</type>
-    <joint name="wheel_RL_joint">
-      <hardwareInterface>hardware_interface/VelocityJointInterface</hardwareInterface>
-    </joint>
-    <actuator name="wheel_RL_actuator">
-      <hardwareInterface>hardware_interface/VelocityJointInterface</hardwareInterface>
-      <mechanicalReduction>1</mechanicalReduction>
-    </actuator>
-  </transmission>
 </robot>

File: aleph2_description/urdf/include/aleph2.gazebo.xacro (robot description, xacro)
@@ -1,4 +1,4 @@
 <?xml version="1.0"?>
-<robot>
+<robot xmlns:xacro="http://www.ros.org/wiki/xacro">
   <!-- ros_control plugin -->
   <gazebo>
@@ -71,3 +71,13 @@
     <selfCollide>true</selfCollide>
   </gazebo>
+  <!-- rocker differential -->
+  <!-- <xacro:unless value="$(arg rockers_fixed)">
+    <gazebo>
+      <plugin name="rocker_differential" filename="libgazebo_differential_plugin.so">
+        <jointA>rocker_L_joint</jointA>
+        <jointB>rocker_R_joint</jointB>
+        <forceConstant>100.0</forceConstant>
+      </plugin>
+    </gazebo>
+  </xacro:unless> -->
 </robot>

File: aleph2_description/urdf/include/manip.urdf.xacro (robot description, xacro)
@@ -1,4 +1,4 @@
 <?xml version="1.0"?>
-<robot>
+<robot xmlns:xacro="http://www.ros.org/wiki/xacro">
   <!-- LINKS -->
   <link name="manip_base_link">

File: aleph2_description/urdf/include/materials.urdf.xacro (robot description, xacro)
@@ -1,4 +1,4 @@
 <?xml version="1.0"?>
-<robot>
+<robot xmlns:xacro="http://www.ros.org/wiki/xacro">
   <material name="base">
     <color rgba="0.3 0.3 0.3 1"/>

File: aleph2_description/urdf/include/zed.urdf.xacro (robot description, xacro)
@@ -1,4 +1,4 @@
 <?xml version="1.0"?>
-<robot>
+<robot xmlns:xacro="http://www.ros.org/wiki/xacro">
   <!-- LINKS -->
   <link name="zed_camera_link">

Commit message: aleph2_description: Add dummy transmissions for rocker joints

File: aleph2_description/urdf/aleph2.urdf.xacro (robot description, xacro)
@@ -136,5 +136,5 @@
     <axis xyz="0 0 1"/>
     <limit effort="100.0" lower="-0.3" upper="0.3" velocity="100.0"/>
-    <dynamics friction="1.0" damping="0.1"/>
+    <dynamics friction="1.0" damping="0.5"/>
   </joint>
   <joint name="rocker_L_joint" type="${rockers_joint_type}">
@@ -144,5 +144,5 @@
     <axis xyz="0 0 1"/>
     <limit effort="100.0" lower="-0.3" upper="0.3" velocity="100.0"/>
-    <dynamics friction="1.0" damping="0.1"/>
+    <dynamics friction="1.0" damping="0.5"/>
   </joint>
   <joint name="mast_joint" type="fixed">
@@ -151,3 +151,21 @@
     <origin xyz="-0.22 0.25 -0.15"/>
   </joint>
+  <!-- TRANSMISSIONS -->
+  <!-- Dummy transmissions for rocker joints -->
+  <xacro:unless value="$(arg rockers_fixed)">
+    <transmission name="rocker_L_trans">
+      <type>transmission_interface/SimpleTransmission</type>
+      <joint name="rocker_L_joint">
+        <hardwareInterface>hardware_interface/EffortJointInterface</hardwareInterface>
+      </joint>
+      <actuator name="rocker_L_virtual_motor"/>
+    </transmission>
+    <transmission name="rocker_R_trans">
+      <type>transmission_interface/SimpleTransmission</type>
+      <joint name="rocker_R_joint">
+        <hardwareInterface>hardware_interface/EffortJointInterface</hardwareInterface>
+      </joint>
+      <actuator name="rocker_R_virtual_motor"/>
+    </transmission>
+  </xacro:unless>
 </robot>

Commit message: Add base_footprint link

File: aleph2_description/urdf/aleph2.urdf.xacro (robot description, xacro)
@@ -18,4 +18,5 @@
   </xacro:if>
   <!-- LINKS -->
+  <link name="base_footprint"/>
   <link name="base_link">
     <visual>
@@ -124,4 +125,9 @@
   </link>
   <!-- JOINTS -->
+  <joint name="base_joint" type="fixed">
+    <origin xyz="0 0 0.33" rpy="0 0 0"/>
+    <parent link="base_footprint"/>
+    <child link="base_link"/>
+  </joint>
   <xacro:if value="$(arg rockers_fixed)">
     <xacro:property name="rockers_joint_type" value="fixed"/>

Commit message: Split configuration, add gazebo_ros2_control

File: aleph2_description/urdf/aleph2.urdf.xacro (robot description, xacro)
@@ -2,158 +2,9 @@
 <robot xmlns:xacro="http://www.ros.org/wiki/xacro"
        name="aleph2">
-  <xacro:arg name="fixed" default="false"/>
   <xacro:arg name="rockers_fixed" default="true"/>
-  <xacro:include filename="$(find aleph2_description)/urdf/include/materials.urdf.xacro" />
-  <xacro:include filename="$(find aleph2_description)/urdf/include/aleph2.gazebo.xacro" />
-  <xacro:include filename="$(find aleph2_description)/urdf/include/drivetrain.urdf.xacro" />
-  <xacro:include filename="$(find aleph2_description)/urdf/include/manip.urdf.xacro" />
-  <xacro:include filename="$(find aleph2_description)/urdf/include/zed.urdf.xacro" />
-  <xacro:if value="$(arg fixed)">
-    <link name="world"/>
-    <joint name="fixed" type="fixed">
-      <parent link="world"/>
-      <child link="base_link"/>
-      <origin xyz="0.0 0.0 2.0"/>
-    </joint>
-  </xacro:if>
-  <!-- LINKS -->
-  <link name="base_footprint"/>
-  <link name="base_link">
-    <visual>
-      <geometry>
-        <mesh filename="package://aleph2_description/models/base.STL" />
-      </geometry>
-      <origin xyz="0 0 0" rpy="${pi/2} 0 ${pi/2}"/>
-      <material name="base" />
-    </visual>
-    <visual>
-      <geometry>
-        <cylinder radius="0.02" length="0.12" />
-      </geometry>
-      <origin xyz="0.06 0.125 0.063" />
-      <material name="motor">
-        <color rgba="0 0 0.5 1"/>
-      </material>
-    </visual>
-    <visual>
-      <geometry>
-        <cylinder radius="0.016" length="0.1" />
-      </geometry>
-      <origin xyz="0.151 0.175 0.053" />
-      <material name="encoder">
-        <color rgba="0 0.5 0 1"/>
-      </material>
-    </visual>
-    <collision>
-      <geometry>
-        <box size="0.72 0.5 0.1"/>
-      </geometry>
-      <origin xyz="-0.08 0 0"/>
-    </collision>
-    <collision>
-      <geometry>
-        <box size="0.16 0.5 0.1"/>
-      </geometry>
-      <origin xyz="-0.06 0 0.09"/>
-    </collision>
-    <collision>
-      <geometry>
-        <cylinder radius="0.02" length="0.12" />
-      </geometry>
-      <origin xyz="0.06 0.125 0.063" />
-    </collision>
-    <collision>
-      <geometry>
-        <cylinder radius="0.016" length="0.1" />
-      </geometry>
-      <origin xyz="0.151 0.175 0.053" />
-    </collision>
-    <inertial>
-      <origin xyz="-0.06700 0.00064 0.00551"/>
-      <mass value="9.0" />
-      <inertia ixx="0.23691" ixy="-0.00014" ixz="-0.00314"
-               iyy="0.23328" iyz="-0.00054" izz="0.40961" />
-    </inertial>
-  </link>
-  <xacro:macro name="rocker" params="name">
-    <link name="rocker_${name}_link">
-      <visual>
-        <geometry>
-          <mesh filename="package://aleph2_description/models/rocker.STL"/>
-        </geometry>
-        <material name="rocker" />
-      </visual>
-      <collision>
-        <geometry>
-          <mesh filename="package://aleph2_description/models/rocker_collision.STL" />
-        </geometry>
-      </collision>
-      <inertial>
-        <origin xyz="0.00000 -0.01737 0.03763"/>
-        <mass value="1.5" />
-        <inertia ixx="0.01934" ixy="-0.00942" ixz="-0.00271"
-                 iyy="0.03716" iyz="0.00516"  izz="0.04409" />
-      </inertial>
-    </link>
-  </xacro:macro>
-  <xacro:rocker name="R" />
-  <xacro:rocker name="L" />
-  <link name="mast_link">
-    <visual>
-      <geometry>
-        <cylinder radius="0.02" length="1.3" />
-      </geometry>
-      <origin xyz="0 0 0.65" rpi="0 0 0"/>
-      <material name="mast" />
-    </visual>
-    <collision>
-      <geometry>
-        <cylinder radius="0.03" length="1.3" />
-      </geometry>
-      <origin xyz="0 0 0.65" rpi="0 0 0"/>
-    </collision>
-    <collision>
-      <geometry>
-        <cylinder radius="0.1" length="0.7" />
-      </geometry>
-      <origin xyz="0 0 0.95" rpi="0 0 0"/>
-    </collision>
-    <inertial>
-      <mass value="1.0" />
-      <inertia ixx="1.0" ixy="0.0" ixz="0.0" iyy="1.0" iyz="0.0" izz="1.0" />
-    </inertial>
-  </link>
-  <!-- JOINTS -->
-  <joint name="base_joint" type="fixed">
-    <origin xyz="0 0 0.33" rpy="0 0 0"/>
-    <parent link="base_footprint"/>
-    <child link="base_link"/>
-  </joint>
-  <xacro:if value="$(arg rockers_fixed)">
-    <xacro:property name="rockers_joint_type" value="fixed"/>
-  </xacro:if>
-  <xacro:unless value="$(arg rockers_fixed)">
-    <xacro:property name="rockers_joint_type" value="revolute"/>
-  </xacro:unless>
-  <joint name="rocker_R_joint" type="${rockers_joint_type}">
-    <parent link="base_link"/>
-    <child link="rocker_R_link"/>
-    <origin xyz="0 -0.375 0" rpy="${pi/2} 0 ${pi}"/>
-    <axis xyz="0 0 1"/>
-    <limit effort="100.0" lower="-0.3" upper="0.3" velocity="100.0"/>
-    <dynamics friction="1.0" damping="0.5"/>
-  </joint>
-  <joint name="rocker_L_joint" type="${rockers_joint_type}">
-    <parent link="base_link"/>
-    <child link="rocker_L_link"/>
-    <origin xyz="0 0.375 0" rpy="${pi/2} 0 0"/>
-    <axis xyz="0 0 1"/>
-    <limit effort="100.0" lower="-0.3" upper="0.3" velocity="100.0"/>
-    <dynamics friction="1.0" damping="0.5"/>
-  </joint>
-  <joint name="mast_joint" type="fixed">
-    <parent link="base_link" />
-    <child link="mast_link" />
-    <origin xyz="-0.22 0.25 -0.15"/>
-  </joint>
+  <xacro:include filename="include/materials.xacro" />
+  <xacro:include filename="include/base.xacro"/>
+  <xacro:include filename="include/drivetrain.xacro" />
+  <xacro:include filename="include/manip.xacro" />
+  <xacro:include filename="include/zed.xacro" />
 </robot>

Commit message: Update description

File: aleph2_description/urdf/aleph2.urdf.xacro (robot description, xacro)
@@ -1,10 +1,11 @@
 <?xml version="1.0"?>
 <robot xmlns:xacro="http://www.ros.org/wiki/xacro"
-       name="aleph2">
-  <xacro:arg name="rockers_fixed" default="true"/>
+  name="aleph2">
+  <xacro:arg name="rockers_fixed" default="true" />
   <xacro:include filename="include/materials.xacro" />
-  <xacro:include filename="include/base.xacro"/>
+  <xacro:include filename="include/base.xacro" />
   <xacro:include filename="include/drivetrain.xacro" />
   <xacro:include filename="include/manip.xacro" />
   <xacro:include filename="include/zed.xacro" />
+  <xacro:include filename="$(find aleph2_description)/ros2_control/aleph2.ros2_control.xacro" />
 </robot>

File: aleph2_description/urdf/include/gazebo.xacro (robot description, xacro)
@@ -81,91 +81,3 @@
     </plugin>
   </gazebo>
-  <ros2_control name="DrivetrainGazeboSystem" type="system">
-    <hardware>
-      <plugin>gazebo_ros2_control/GazeboSystem</plugin>
-    </hardware>
-    <joint name="rocker_L_joint">
-      <state_interface name="position"/>
-    </joint>
-    <joint name="rocker_R_joint">
-      <state_interface name="position"/>
-    </joint>
-    <joint name="wheel_FL_joint">
-      <command_interface name="velocity"/>
-      <state_interface name="position"/>
-      <state_interface name="velocity"/>
-      <state_interface name="effort"/>
-    </joint>
-    <joint name="wheel_RL_joint">
-      <command_interface name="velocity"/>
-      <state_interface name="position"/>
-      <state_interface name="velocity"/>
-      <state_interface name="effort"/>
-    </joint>
-    <joint name="wheel_FR_joint">
-      <command_interface name="velocity"/>
-      <state_interface name="position"/>
-      <state_interface name="velocity"/>
-      <state_interface name="effort"/>
-    </joint>
-    <joint name="wheel_RR_joint">
-      <command_interface name="velocity"/>
-      <state_interface name="position"/>
-      <state_interface name="velocity"/>
-      <state_interface name="effort"/>
-    </joint>
-  </ros2_control>
-  <ros2_control name="ManipGazeboSystem" type="system">
-    <hardware>
-      <plugin>gazebo_ros2_control/GazeboSystem</plugin>
-    </hardware>
-    <joint name="manip_base_joint">
-      <command_interface name="position"/>
-      <command_interface name="velocity"/>
-      <command_interface name="effort"/>
-      <state_interface name="position"/>
-      <state_interface name="velocity"/>
-      <state_interface name="effort"/>
-    </joint>
-    <joint name="manip_shoulder_joint">
-      <command_interface name="position"/>
-      <command_interface name="velocity"/>
-      <command_interface name="effort"/>
-      <state_interface name="position"/>
-      <state_interface name="velocity"/>
-      <state_interface name="effort"/>
-    </joint>
-    <joint name="manip_elbow_joint">
-      <command_interface name="position"/>
-      <command_interface name="velocity"/>
-      <command_interface name="effort"/>
-      <state_interface name="position"/>
-      <state_interface name="velocity"/>
-      <state_interface name="effort"/>
-    </joint>
-    <joint name="manip_wrist_tilt_joint">
-      <command_interface name="position"/>
-      <command_interface name="velocity"/>
-      <command_interface name="effort"/>
-      <state_interface name="position"/>
-      <state_interface name="velocity"/>
-      <state_interface name="effort"/>
-    </joint>
-    <joint name="manip_wrist_roll_joint">
-      <command_interface name="position"/>
-      <command_interface name="velocity"/>
-      <command_interface name="effort"/>
-      <state_interface name="position"/>
-      <state_interface name="velocity"/>
-      <state_interface name="effort"/>
-    </joint>
-    <joint name="manip_gripper_joint">
-      <command_interface name="position"/>
-      <command_interface name="velocity"/>
-      <command_interface name="effort"/>
-      <state_interface name="position"/>
-      <state_interface name="velocity"/>
-      <state_interface name="effort"/>
-    </joint>
-  </ros2_control>
 </robot>
