Commit message: Disable components which are not needed for now

File: aleph2_description/urdf/aleph2_sim.urdf.xacro (robot description, xacro)
@@ -7,5 +7,5 @@
   <xacro:include filename="include/base.xacro" />
   <xacro:include filename="include/drivetrain.xacro" />
-  <xacro:include filename="include/manip.xacro" />
+  <!-- <xacro:include filename="include/manip.xacro" /> -->
   <xacro:include filename="include/zed.xacro" />
   <xacro:include filename="include/gazebo.xacro" />

File: aleph2_description/urdf/include/base.xacro (robot description, xacro)
@@ -83,5 +83,5 @@
   <xacro:rocker name="R" />
   <xacro:rocker name="L" />
-  <link name="mast_link">
+  <!-- <link name="mast_link">
     <visual>
       <geometry>
@@ -107,5 +107,5 @@
       <inertia ixx="1.0" ixy="0.0" ixz="0.0" iyy="1.0" iyz="0.0" izz="1.0" />
     </inertial>
-  </link>
+  </link> -->
   <!-- JOINTS -->
   <joint name="base_joint" type="fixed">
@@ -136,8 +136,8 @@
     <dynamics friction="1.0" damping="0.5"/>
   </joint>
-  <joint name="mast_joint" type="fixed">
+  <!-- <joint name="mast_joint" type="fixed">
     <parent link="base_link" />
     <child link="mast_link" />
     <origin xyz="-0.22 0.25 -0.15"/>
-  </joint>
+  </joint> -->
 </robot>
