Commit message: Update ros2_control urdf tag

File: aleph2_description/ros2_control/aleph2.ros2_control.xacro (robot description, xacro)
@@ -1,31 +1,22 @@
 <?xml version="1.0"?>
 <robot xmlns:xacro="http://www.ros.org/wiki/xacro">
-  <ros2_control name="DrivetrainSystem" type="system">
+  <ros2_control name="NanotecSystem" type="system">
     <hardware>
-      <plugin>aleph2_hardware/Aleph2NanotecSystem</plugin>
+      <plugin>nanotec_driver/NanotecSystem</plugin>
+      <param name="can_interface_name">can0</param>
+      <param name="bus_config_package">aleph2_bringup</param>
+      <param name="bus_config_name">nanotec_bus</param>
     </hardware>
+    <joint name="wheel_RR_joint">
+      <param name="node_id">1</param>
+    </joint>
+    <joint name="wheel_FR_joint">
+      <param name="node_id">2</param>
+    </joint>
     <joint name="wheel_FL_joint">
-      <command_interface name="velocity" />
-      <state_interface name="position" />
-      <state_interface name="velocity" />
-      <state_interface name="effort" />
+      <param name="node_id">3</param>
     </joint>
     <joint name="wheel_RL_joint">
-      <command_interface name="velocity" />
-      <state_interface name="position" />
-      <state_interface name="velocity" />
-      <state_interface name="effort" />
-    </joint>
-    <joint name="wheel_FR_joint">
-      <command_interface name="velocity" />
-      <state_interface name="position" />
-      <state_interface name="velocity" />
-      <state_interface name="effort" />
-    </joint>
-    <joint name="wheel_RR_joint">
-      <command_interface name="velocity" />
-      <state_interface name="position" />
-      <state_interface name="velocity" />
-      <state_interface name="effort" />
+      <param name="node_id">4</param>
     </joint>
   </ros2_control>
